File: pcb/vagrant.kicad_pcb (KiCad board)
At the start: 2 copper layers, 83.8 x 90.2 mm, 30 parts, among them K1 KEYSW, K10 KEYSW, K2 KEYSW, K3 KEYSW, K4 KEYSW, K5 KEYSW, K6 KEYSW, K7 KEYSW, K8 KEYSW, K9 KEYSW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

Commit message: added Readme
Parts:
- added HOLE_M3: VAL**, keyboard_parts:HOLE_M3, F.Cu at (136.5, 36.8)
- added HOLE_M3: VAL**, keyboard_parts:HOLE_M3, F.Cu at (110.5, 74.9)
- added HOLE_M3: VAL**, keyboard_parts:HOLE_M3, F.Cu at (136.5, 114.3)
- added HOLE_M3: VAL**, keyboard_parts:HOLE_M3, F.Cu at (65.4, 36.8)
- added HOLE_M3: VAL**, keyboard_parts:HOLE_M3, F.Cu at (65.4, 114.3)
- G***: moved to B.Cu
- moved G*** 92.1 mm to (97.8, 75.6), turned to 180 degrees
Other:
- board size 83.8 x 90.2 mm -> 169.5 x 90.2 mm
